File: _saved_audio_input.sch (KiCad schematic (older format))
At the start: 17 parts, among them U8 OPA1664

Commit message: Fixed decoupling cap polarity on output op-amp, added bias to analog input, changed capacitor footprints to reflect new capacitor selections
Other:
- note added: "Design referenced from PCM3060\ndatasheet P40 (SLAS533B)"
Changed lines of the file:
@@
 Text Notes 7600 3050 0    60   ~ 0
 Input biased by VCOM \nwhere VCOM = VCC/2 (2.5V nom.)
+Text Notes 6350 7000 0    60   ~ 0
+Design referenced from PCM3060\ndatasheet P40 (SLAS533B)
 $EndSCHEMATC
