File: audio_output.sch (KiCad schematic (older format))
At the start: 26 parts

Commit message: Added annotations, fixed ERC errors
Parts:
- gave numbers to parts that had none: 25
Changed lines of the file:
@@
 $EndDescr
 $Comp
-L OPA1664 U?
+L OPA1664 U9
 U 3 1 5A4A0205
 P 5250 2050
-F 0 "U?" H 5300 2250 60  0000 C CNN
+F 0 "U9" H 5300 2250 60  0000 C CNN
 F 1 "OPA1664" H 5400 1850 50  0000 C CNN
 F 2 "" H 5250 2050 60  0000 C CNN
@@
 	5150 1500 5150 1650
 $Comp
-L -5V #PWR?
+L -5V #PWR076
 U 1 1 5A4A0210
 P 6500 1500
-F 0 "#PWR?" H 6500 1640 20  0001 C CNN
+F 0 "#PWR076" H 6500 1640 20  0001 C CNN
 F 1 "-5V" H 6500 1610 30  0000 C CNN
 F 2 "" H 6500 1500 60  0000 C CNN
@@
 $EndComp
 $Comp
-L +5V #PWR?
+L +5V #PWR077
 U 1 1 5A4A0216
 P 6500 2650
-F 0 "#PWR?" H 6500 2740 20  0001 C CNN
+F 0 "#PWR077" H 6500 2740 20  0001 C CNN
 F 1 "+5V" H 6500 2740 30  0000 C CNN
 F 2 "" H 6500 2650 60  0000 C CNN
@@
 	5150 2450 5150 2800
 $Comp
-L C C?
+L C C31
 U 1 1 5A4A021E
 P 5150 1200
-F 0 "C?" V 5200 1300 50  0000 L CNN
+F 0 "C31" V 5200 1300 50  0000 L CNN
 F 1 "470pF" V 5200 900 50  0000 L CNN
 F 2 "" H 5150 1200 60  0000 C CNN
@@
 Connection ~ 4700 1950
 $Comp
-L CP1 C?
+L CP1 C34
 U 1 1 5A4A0239
 P 5150 3000
-F 0 "C?" H 5200 3100 50  0000 L CNN
+F 0 "C34" H 5200 3100 50  0000 L CNN
 F 1 "CP1" H 5200 2900 50  0000 L CNN
 F 2 "" H 5150 3000 60  0000 C CNN
@@
 	5850 1200 5350 1200
 $Comp
-L R R?
+L R R30
 U 1 1 5A4A0249
 P 5150 850
-F 0 "R?" H 4950 900 50  0000 C CNN
+F 0 "R30" H 4950 900 50  0000 C CNN
 F 1 "7.5k" H 5350 900 50  0000 C CNN
 F 2 "" H 5150 850 60  0000 C CNN
@@
 Connection ~ 5850 1200
 $Comp
-L CP1 C?
+L CP1 C35
 U 1 1 5A4A0254
 P 6200 3000
-F 0 "C?" H 6250 3100 50  0000 L CNN
+F 0 "C35" H 6250 3100 50  0000 L CNN
 F 1 "CP1" H 6250 2900 50  0000 L CNN
 F 2 "" H 6200 3000 60  0000 C CNN
@@
 Connection ~ 6200 1500
 $Comp
-L GND #PWR?
+L GND #PWR078
 U 1 1 5A4A0265
 P 5150 3400
-F 0 "#PWR?" H 5150 3400 30  0001 C CNN
+F 0 "#PWR078" H 5150 3400 30  0001 C CNN
 F 1 "GND" H 5150 3330 30  0001 C CNN
 F 2 "" H 5150 3400 60  0000 C CNN
@@
 	5150 3400 5150 3200
 $Comp
-L GND #PWR?
+L GND #PWR079
 U 1 1 5A4A026C
 P 6200 3400
-F 0 "#PWR?" H 6200 3400 30  0001 C CNN
+F 0 "#PWR079" H 6200 3400 30  0001 C CNN
 F 1 "GND" H 6200 3330 30  0001 C CNN
 F 2 "" H 6200 3400 60  0000 C CNN
@@
 	6200 3400 6200 3200
 $Comp
-L R R?
+L R R32
 U 1 1 5A4A0273
 P 4350 1950
-F 0 "R?" H 4150 2000 50  0000 C CNN
+F 0 "R32" H 4150 2000 50  0000 C CNN
 F 1 "820" H 4550 2000 50  0000 C CNN
 F 2 "" H 4350 1950 60  0000 C CNN
@@
 $EndComp
 $Comp
-L R R?
+L R R33
 U 1 1 5A4A027B
 P 6650 2050
-F 0 "R?" H 6450 2100 50  0000 C CNN
+F 0 "R33" H 6450 2100 50  0000 C CNN
 F 1 "100" H 6850 2100 50  0000 C CNN
 F 2 "" H 6650 2050 60  0000 C CNN
@@
 	7250 2050 6850 2050
 $Comp
-L R R?
+L R R34
 U 1 1 5A4A0409
 P 4350 2150
-F 0 "R?" H 4150 2200 50  0000 C CNN
+F 0 "R34" H 4150 2200 50  0000 C CNN
 F 1 "820" H 4550 2200 50  0000 C CNN
 F 2 "" H 4350 2150 60  0000 C CNN
@@
 $EndComp
 $Comp
-L C C?
+L C C33
 U 1 1 5A4A043D
 P 4700 3000
-F 0 "C?" H 4750 3100 50  0000 L CNN
+F 0 "C33" H 4750 3100 50  0000 L CNN
 F 1 "470pF" H 4750 2900 50  0000 L CNN
 F 2 "" H 4700 3000 60  0000 C CNN
@@
 $EndComp
 $Comp
-L GND #PWR?
+L GND #PWR080
 U 1 1 5A4A0477
 P 4700 3400
-F 0 "#PWR?" H 4700 3400 30  0001 C CNN
+F 0 "#PWR080" H 4700 3400 30  0001 C CNN
 F 1 "GND" H 4700 3330 30  0001 C CNN
 F 2 "" H 4700 3400 60  0000 C CNN
@@
 Connection ~ 4700 2150
 $Comp
-L C C?
+L C C32
 U 1 1 5A4A05D6
 P 3550 2150
-F 0 "C?" V 3600 2250 50  0000 L CNN
+F 0 "C32" V 3600 2250 50  0000 L CNN
 F 1 "1500pF" V 3600 1800 50  0000 L CNN
 F 2 "" H 3550 2150 60  0000 C CNN
@@
 	3100 1950 4150 1950
 $Comp
-L R R?
+L R R31
 U 1 1 5A4A064B
 P 2900 1950
-F 0 "R?" H 2700 2000 50  0000 C CNN
+F 0 "R31" H 2700 2000 50  0000 C CNN
 F 1 "10k" H 3100 2000 50  0000 C CNN
 F 2 "" H 2900 1950 60  0000 C CNN
@@
 Connection ~ 4000 2150
 $Comp
-L R R?
+L R R35
 U 1 1 5A4A07FE
 P 2900 2350
-F 0 "R?" H 2700 2400 50  0000 C CNN
+F 0 "R35" H 2700 2400 50  0000 C CNN
 F 1 "10k" H 3100 2400 50  0000 C CNN
 F 2 "" H 2900 2350 60  0000 C CNN
@@
 	4000 2150 4000 2750
 $Comp
-L R R?
+L R R36
 U 1 1 5A4A0B17
 P 4000 2950
-F 0 "R?" V 3800 3000 50  0000 C CNN
+F 0 "R36" V 3800 3000 50  0000 C CNN
 F 1 "7.5K" V 4200 3050 50  0000 C CNN
 F 2 "" H 4000 2950 60  0000 C CNN
@@
 Connection ~ 4000 2350
 $Comp
-L GND #PWR?
+L GND #PWR081
 U 1 1 5A4A0BAE
 P 4000 3400
-F 0 "#PWR?" H 4000 3400 30  0001 C CNN
+F 0 "#PWR081" H 4000 3400 30  0001 C CNN
 F 1 "GND" H 4000 3330 30  0001 C CNN
 F 2 "" H 4000 3400 60  0000 C CNN
@@
 	4000 3400 4000 3150
 $Comp
-L OPA1664 U?
+L OPA1664 U9
 U 4 1 5A4A115F
 P 5300 5000
-F 0 "U?" H 5350 5200 60  0000 C CNN
+F 0 "U9" H 5350 5200 60  0000 C CNN
 F 1 "OPA1664" H 5450 4800 50  0000 C CNN
 F 2 "" H 5300 5000 60  0000 C CNN
@@
 	5200 4450 5200 4600
 $Comp
-L -5V #PWR?
+L -5V #PWR082
 U 1 1 5A4A1169
 P 6550 4450
-F 0 "#PWR?" H 6550 4590 20  0001 C CNN
+F 0 "#PWR082" H 6550 4590 20  0001 C CNN
 F 1 "-5V" H 6550 4560 30  0000 C CNN
 F 2 "" H 6550 4450 60  0000 C CNN
@@
 $EndComp
 $Comp
-L +5V #PWR?
+L +5V #PWR083
 U 1 1 5A4A116F
 P 6550 5600
-F 0 "#PWR?" H 6550 5690 20  0001 C CNN
+F 0 "#PWR083" H 6550 5690 20  0001 C CNN
 F 1 "+5V" H 6550 5690 30  0000 C CNN
 F 2 "" H 6550 5600 60  0000 C CNN
@@
 	5200 5400 5200 5750
 $Comp
-L C C?
+L C C36
 U 1 1 5A4A1176
 P 5200 4150
-F 0 "C?" V 5250 4250 50  0000 L CNN
+F 0 "C36" V 5250 4250 50  0000 L CNN
 F 1 "470pF" V 5250 3850 50  0000 L CNN
 F 2 "" H 5200 4150 60  0000 C CNN
@@
 Connection ~ 4750 4900
 $Comp
-L CP1 C?
+L CP1 C39
 U 1 1 5A4A117E
 P 5200 5950
-F 0 "C?" H 5250 6050 50  0000 L CNN
+F 0 "C39" H 5250 6050 50  0000 L CNN
 F 1 "CP1" H 5250 5850 50  0000 L CNN
 F 2 "" H 5200 5950 60  0000 C CNN
@@
 	5900 4150 5400 4150
 $Comp
-L R R?
+L R R37
 U 1 1 5A4A118B
 P 5200 3800
-F 0 "R?" H 5000 3850 50  0000 C CNN
+F 0 "R37" H 5000 3850 50  0000 C CNN
 F 1 "7.5k" H 5400 3850 50  0000 C CNN
 F 2 "" H 5200 3800 60  0000 C CNN
@@
 Connection ~ 5900 4150
 $Comp
-L CP1 C?
+L CP1 C40
 U 1 1 5A4A1194
 P 6250 5950
-F 0 "C?" H 6300 6050 50  0000 L CNN
+F 0 "C40" H 6300 6050 50  0000 L CNN
 F 1 "CP1" H 6300 5850 50  0000 L CNN
 F 2 "" H 6250 5950 60  0000 C CNN
@@
 Connection ~ 6250 4450
 $Comp
-L GND #PWR?
+L GND #PWR084
 U 1 1 5A4A119D
 P 5200 6350
-F 0 "#PWR?" H 5200 6350 30  0001 C CNN
+F 0 "#PWR084" H 5200 6350 30  0001 C CNN
 F 1 "GND" H 5200 6280 30  0001 C CNN
 F 2 "" H 5200 6350 60  0000 C CNN
@@
 	5200 6350 5200 6150
 $Comp
-L GND #PWR?
+L GND #PWR085
 U 1 1 5A4A11A4
 P 6250 6350
-F 0 "#PWR?" H 6250 6350 30  0001 C CNN
+F 0 "#PWR085" H 6250 6350 30  0001 C CNN
 F 1 "GND" H 6250 6280 30  0001 C CNN
 F 2 "" H 6250 6350 60  0000 C CNN
@@
 	6250 6350 6250 6150
 $Comp
-L R R?
+L R R39
 U 1 1 5A4A11AB
 P 4400 4900
-F 0 "R?" H 4200 4950 50  0000 C CNN
+F 0 "R39" H 4200 4950 50  0000 C CNN
 F 1 "820" H 4600 4950 50  0000 C CNN
 F 2 "" H 4400 4900 60  0000 C CNN
@@
 $EndComp
 $Comp
-L R R?
+L R R40
 U 1 1 5A4A11B2
 P 6700 5000
-F 0 "R?" H 6500 5050 50  0000 C CNN
+F 0 "R40" H 6500 5050 50  0000 C CNN
 F 1 "100" H 6900 5050 50  0000 C CNN
 F 2 "" H 6700 5000 60  0000 C CNN
@@
 	7300 5000 6900 5000
 $Comp
-L R R?
+L R R41
 U 1 1 5A4A11BD
 P 4400 5100
-F 0 "R?" H 4200 5150 50  0000 C CNN
+F 0 "R41" H 4200 5150 50  0000 C CNN
 F 1 "820" H 4600 5150 50  0000 C CNN
 F 2 "" H 4400 5100 60  0000 C CNN
@@
 $EndComp
 $Comp
-L C C?
+L C C38
 U 1 1 5A4A11C4
 P 4750 5950
-F 0 "C?" H 4800 6050 50  0000 L CNN
+F 0 "C38" H 4800 6050 50  0000 L CNN
 F 1 "470pF" H 4800 5850 50  0000 L CNN
 F 2 "" H 4750 5950 60  0000 C CNN
@@
 $EndComp
 $Comp
-L GND #PWR?
+L GND #PWR086
 U 1 1 5A4A11CB
 P 4750 6350
-F 0 "#PWR?" H 4750 6350 30  0001 C CNN
+F 0 "#PWR086" H 4750 6350 30  0001 C CNN
 F 1 "GND" H 4750 6280 30  0001 C CNN
 F 2 "" H 4750 6350 60  0000 C CNN
@@
 Connection ~ 4750 5100
 $Comp
-L C C?
+L C C37
 U 1 1 5A4A11D5
 P 3600 5100
-F 0 "C?" V 3650 5200 50  0000 L CNN
+F 0 "C37" V 3650 5200 50  0000 L CNN
 F 1 "1500pF" V 3650 4750 50  0000 L CNN
 F 2 "" H 3600 5100 60  0000 C CNN
@@
 	3150 4900 4200 4900
 $Comp
-L R R?
+L R R38
 U 1 1 5A4A11DD
 P 2950 4900
-F 0 "R?" H 2750 4950 50  0000 C CNN
+F 0 "R38" H 2750 4950 50  0000 C CNN
 F 1 "10k" H 3150 4950 50  0000 C CNN
 F 2 "" H 2950 4900 60  0000 C CNN
@@
 Connection ~ 4050 5100
 $Comp
-L R R?
+L R R42
 U 1 1 5A4A11EA
 P 2950 5300
-F 0 "R?" H 2750 5350 50  0000 C CNN
+F 0 "R42" H 2750 5350 50  0000 C CNN
 F 1 "10k" H 3150 5350 50  0000 C CNN
 F 2 "" H 2950 5300 60  0000 C CNN
@@
 	4050 5100 4050 5700
 $Comp
-L R R?
+L R R43
 U 1 1 5A4A11F9
 P 4050 5900
-F 0 "R?" V 3850 5950 50  0000 C CNN
+F 0 "R43" V 3850 5950 50  0000 C CNN
 F 1 "7.5K" V 4250 6000 50  0000 C CNN
 F 2 "" H 4050 5900 60  0000 C CNN
@@
 Connection ~ 4050 5300
 $Comp
-L GND #PWR?
+L GND #PWR087
 U 1 1 5A4A1201
 P 4050 6350
-F 0 "#PWR?" H 4050 6350 30  0001 C CNN
+F 0 "#PWR087" H 4050 6350 30  0001 C CNN
 F 1 "GND" H 4050 6280 30  0001 C CNN
 F 2 "" H 4050 6350 60  0000 C CNN

Commit message: Updated decoupling capacitors for op-amp output
Parts:
- removed C34, C35, C39, C40: CP1, symbol CP1
- renumbered C31 to C35, C32 to C36, C33 to C37, C36 to C38, C37 to C39, C38 to C40
Changed lines of the file:
@@
 	5150 1500 5150 1650
 $Comp
-L -5V #PWR078
+L -5V #PWR085
 U 1 1 5A4A0210
 P 6500 1500
-F 0 "#PWR078" H 6500 1640 20  0001 C CNN
+F 0 "#PWR085" H 6500 1640 20  0001 C CNN
 F 1 "-5V" H 6500 1610 30  0000 C CNN
 F 2 "" H 6500 1500 60  0000 C CNN
@@
 $EndComp
 $Comp
-L +5V #PWR079
+L +5V #PWR086
 U 1 1 5A4A0216
 P 6500 2650
-F 0 "#PWR079" H 6500 2740 20  0001 C CNN
+F 0 "#PWR086" H 6500 2740 20  0001 C CNN
 F 1 "+5V" H 6500 2740 30  0000 C CNN
 F 2 "" H 6500 2650 60  0000 C CNN
@@
 	0    1    1    0
 $EndComp
-Wire Wire Line
-	5150 2450 5150 2800
-$Comp
-L C C31
+$Comp
+L C C35
 U 1 1 5A4A021E
 P 5150 1200
-F 0 "C31" V 5200 1300 50  0000 L CNN
+F 0 "C35" V 5200 1300 50  0000 L CNN
 F 1 "470pF" V 5200 900 50  0000 L CNN
 F 2 "" H 5150 1200 60  0000 C CNN
@@
 $EndComp
 Connection ~ 4700 1950
-$Comp
-L CP1 C34
-U 1 1 5A4A0239
-P 5150 3000
-F 0 "C34" H 5200 3100 50  0000 L CNN
-F 1 "CP1" H 5200 2900 50  0000 L CNN
-F 2 "" H 5150 3000 60  0000 C CNN
-F 3 "" H 5150 3000 60  0000 C CNN
-	1    5150 3000
-	1    0    0    -1
-$EndComp
 Wire Wire Line
 	5150 2650 6500 2650
-Connection ~ 5150 2650
 Wire Wire Line
 	5150 1500 6500 1500
@@
 Connection ~ 5850 1200
 $Comp
-L CP1 C35
-U 1 1 5A4A0254
-P 6200 3000
-F 0 "C35" H 6250 3100 50  0000 L CNN
-F 1 "CP1" H 6250 2900 50  0000 L CNN
-F 2 "" H 6200 3000 60  0000 C CNN
-F 3 "" H 6200 3000 60  0000 C CNN
-	1    6200 3000
-	-1   0    0    1
-$EndComp
-Wire Wire Line
-	6200 2800 6200 1500
-Connection ~ 6200 1500
-$Comp
-L GND #PWR080
-U 1 1 5A4A0265
-P 5150 3400
-F 0 "#PWR080" H 5150 3400 30  0001 C CNN
-F 1 "GND" H 5150 3330 30  0001 C CNN
-F 2 "" H 5150 3400 60  0000 C CNN
-F 3 "" H 5150 3400 60  0000 C CNN
-	1    5150 3400
-	1    0    0    -1
-$EndComp
-Wire Wire Line
-	5150 3400 5150 3200
-$Comp
-L GND #PWR081
-U 1 1 5A4A026C
-P 6200 3400
-F 0 "#PWR081" H 6200 3400 30  0001 C CNN
-F 1 "GND" H 6200 3330 30  0001 C CNN
-F 2 "" H 6200 3400 60  0000 C CNN
-F 3 "" H 6200 3400 60  0000 C CNN
-	1    6200 3400
-	1    0    0    -1
-$EndComp
-Wire Wire Line
-	6200 3400 6200 3200
-$Comp
 L R R32
 U 1 1 5A4A0273
@@
 $EndComp
 $Comp
-L C C33
+L C C37
 U 1 1 5A4A043D
 P 4700 3000
-F 0 "C33" H 4750 3100 50  0000 L CNN
+F 0 "C37" H 4750 3100 50  0000 L CNN
 F 1 "470pF" H 4750 2900 50  0000 L CNN
 F 2 "" H 4700 3000 60  0000 C CNN
@@
 $EndComp
 $Comp
-L GND #PWR082
+L GND #PWR087
 U 1 1 5A4A0477
 P 4700 3400
-F 0 "#PWR082" H 4700 3400 30  0001 C CNN
+F 0 "#PWR087" H 4700 3400 30  0001 C CNN
 F 1 "GND" H 4700 3330 30  0001 C CNN
 F 2 "" H 4700 3400 60  0000 C CNN
@@
 Connection ~ 4700 2150
 $Comp
-L C C32
+L C C36
 U 1 1 5A4A05D6
 P 3550 2150
-F 0 "C32" V 3600 2250 50  0000 L CNN
+F 0 "C36" V 3600 2250 50  0000 L CNN
 F 1 "1500pF" V 3600 1800 50  0000 L CNN
 F 2 "" H 3550 2150 60  0000 C CNN
@@
 Connection ~ 4000 2350
 $Comp
-L GND #PWR083
+L GND #PWR088
 U 1 1 5A4A0BAE
 P 4000 3400
-F 0 "#PWR083" H 4000 3400 30  0001 C CNN
+F 0 "#PWR088" H 4000 3400 30  0001 C CNN
 F 1 "GND" H 4000 3330 30  0001 C CNN
 F 2 "" H 4000 3400 60  0000 C CNN
@@
 	5200 4450 5200 4600
 $Comp
-L -5V #PWR084
+L -5V #PWR089
 U 1 1 5A4A1169
 P 6550 4450
-F 0 "#PWR084" H 6550 4590 20  0001 C CNN
+F 0 "#PWR089" H 6550 4590 20  0001 C CNN
 F 1 "-5V" H 6550 4560 30  0000 C CNN
 F 2 "" H 6550 4450 60  0000 C CNN
@@
 $EndComp
 $Comp
-L +5V #PWR085
+L +5V #PWR090
 U 1 1 5A4A116F
 P 6550 5600
-F 0 "#PWR085" H 6550 5690 20  0001 C CNN
+F 0 "#PWR090" H 6550 5690 20  0001 C CNN
 F 1 "+5V" H 6550 5690 30  0000 C CNN
 F 2 "" H 6550 5600 60  0000 C CNN
@@
 	0    1    1    0
 $EndComp
-Wire Wire Line
-	5200 5400 5200 5750
-$Comp
-L C C36
+$Comp
+L C C38
 U 1 1 5A4A1176
 P 5200 4150
-F 0 "C36" V 5250 4250 50  0000 L CNN
+F 0 "C38" V 5250 4250 50  0000 L CNN
 F 1 "470pF" V 5250 3850 50  0000 L CNN
 F 2 "" H 5200 4150 60  0000 C CNN
@@
 $EndComp
 Connection ~ 4750 4900
-$Comp
-L CP1 C39
-U 1 1 5A4A117E
-P 5200 5950
-F 0 "C39" H 5250 6050 50  0000 L CNN
-F 1 "CP1" H 5250 5850 50  0000 L CNN
-F 2 "" H 5200 5950 60  0000 C CNN
-F 3 "" H 5200 5950 60  0000 C CNN
-	1    5200 5950
-	1    0    0    -1
-$EndComp
 Wire Wire Line
 	5200 5600 6550 5600
-Connection ~ 5200 5600
 Wire Wire Line
 	5200 4450 6550 4450
@@
 Connection ~ 5900 4150
 $Comp
-L CP1 C40
-U 1 1 5A4A1194
-P 6250 5950
-F 0 "C40" H 6300 6050 50  0000 L CNN
-F 1 "CP1" H 6300 5850 50  0000 L CNN
-F 2 "" H 6250 5950 60  0000 C CNN
-F 3 "" H 6250 5950 60  0000 C CNN
-	1    6250 5950
-	-1   0    0    1
-$EndComp
-Wire Wire Line
-	6250 5750 6250 4450
-Connection ~ 6250 4450
-$Comp
-L GND #PWR086
-U 1 1 5A4A119D
-P 5200 6350
-F 0 "#PWR086" H 5200 6350 30  0001 C CNN
-F 1 "GND" H 5200 6280 30  0001 C CNN
-F 2 "" H 5200 6350 60  0000 C CNN
-F 3 "" H 5200 6350 60  0000 C CNN
-	1    5200 6350
-	1    0    0    -1
-$EndComp
-Wire Wire Line
-	5200 6350 5200 6150
-$Comp
-L GND #PWR087
-U 1 1 5A4A11A4
-P 6250 6350
-F 0 "#PWR087" H 6250 6350 30  0001 C CNN
-F 1 "GND" H 6250 6280 30  0001 C CNN
-F 2 "" H 6250 6350 60  0000 C CNN
-F 3 "" H 6250 6350 60  0000 C CNN
-	1    6250 6350
-	1    0    0    -1
-$EndComp
-Wire Wire Line
-	6250 6350 6250 6150
-$Comp
 L R R39
 U 1 1 5A4A11AB
@@
 $EndComp
 $Comp
-L C C38
+L C C40
 U 1 1 5A4A11C4
 P 4750 5950
-F 0 "C38" H 4800 6050 50  0000 L CNN
+F 0 "C40" H 4800 6050 50  0000 L CNN
 F 1 "470pF" H 4800 5850 50  0000 L CNN
 F 2 "" H 4750 5950 60  0000 C CNN
@@
 $EndComp
 $Comp
-L GND #PWR088
+L GND #PWR091
 U 1 1 5A4A11CB
 P 4750 6350
-F 0 "#PWR088" H 4750 6350 30  0001 C CNN
+F 0 "#PWR091" H 4750 6350 30  0001 C CNN
 F 1 "GND" H 4750 6280 30  0001 C CNN
 F 2 "" H 4750 6350 60  0000 C CNN
@@
 Connection ~ 4750 5100
 $Comp
-L C C37
+L C C39
 U 1 1 5A4A11D5
 P 3600 5100
-F 0 "C37" V 3650 5200 50  0000 L CNN
+F 0 "C39" V 3650 5200 50  0000 L CNN
 F 1 "1500pF" V 3650 4750 50  0000 L CNN
 F 2 "" H 3600 5100 60  0000 C CNN
@@
 Connection ~ 4050 5300
 $Comp
-L GND #PWR089
+L GND #PWR092
 U 1 1 5A4A1201
 P 4050 6350
-F 0 "#PWR089" H 4050 6350 30  0001 C CNN
+F 0 "#PWR092" H 4050 6350 30  0001 C CNN
 F 1 "GND" H 4050 6280 30  0001 C CNN
 F 2 "" H 4050 6350 60  0000 C CNN
@@
 Wire Wire Line
 	4050 6350 4050 6100
+Wire Wire Line
+	5200 5400 5200 5600
+Wire Wire Line
+	5150 2450 5150 2650
 $EndSCHEMATC

Commit message: Added EMI and ESD protection to audio interface, started assoc. footprints
Parts:
- renumbered U9 to U8
Changed lines of the file:
@@
 $EndDescr
 $Comp
-L OPA1664 U9
+L OPA1664 U8
 U 3 1 5A4A0205
 P 5250 2050
-F 0 "U9" H 5300 2250 60  0000 C CNN
+F 0 "U8" H 5300 2250 60  0000 C CNN
 F 1 "OPA1664" H 5400 1850 50  0000 C CNN
-F 2 "" H 5250 2050 60  0000 C CNN
+F 2 "" H 5250 2050 60  0001 C CNN
 F 3 "" H 5250 2050 60  0000 C CNN
 	3    5250 2050
@@
 	5150 1500 5150 1650
 $Comp
-L -5V #PWR085
+L -5V #PWR97
 U 1 1 5A4A0210
 P 6500 1500
-F 0 "#PWR085" H 6500 1640 20  0001 C CNN
+F 0 "#PWR97" H 6500 1640 20  0001 C CNN
 F 1 "-5V" H 6500 1610 30  0000 C CNN
 F 2 "" H 6500 1500 60  0000 C CNN
@@
 $EndComp
 $Comp
-L +5V #PWR086
+L +5V #PWR98
 U 1 1 5A4A0216
 P 6500 2650
-F 0 "#PWR086" H 6500 2740 20  0001 C CNN
+F 0 "#PWR98" H 6500 2740 20  0001 C CNN
 F 1 "+5V" H 6500 2740 30  0000 C CNN
 F 2 "" H 6500 2650 60  0000 C CNN
@@
 F 0 "C35" V 5200 1300 50  0000 L CNN
 F 1 "470pF" V 5200 900 50  0000 L CNN
-F 2 "" H 5150 1200 60  0000 C CNN
+F 2 "" H 5150 1200 60  0001 C CNN
 F 3 "" H 5150 1200 60  0000 C CNN
 	1    5150 1200
@@
 F 0 "R30" H 4950 900 50  0000 C CNN
 F 1 "7.5k" H 5350 900 50  0000 C CNN
-F 2 "" H 5150 850 60  0000 C CNN
+F 2 "" H 5150 850 60  0001 C CNN
 F 3 "" H 5150 850 60  0000 C CNN
 	1    5150 850
@@
 F 0 "R32" H 4150 2000 50  0000 C CNN
 F 1 "820" H 4550 2000 50  0000 C CNN
-F 2 "" H 4350 1950 60  0000 C CNN
+F 2 "" H 4350 1950 60  0001 C CNN
 F 3 "" H 4350 1950 60  0000 C CNN
 	1    4350 1950
@@
 F 0 "R33" H 6450 2100 50  0000 C CNN
 F 1 "100" H 6850 2100 50  0000 C CNN
-F 2 "" H 6650 2050 60  0000 C CNN
+F 2 "" H 6650 2050 60  0001 C CNN
 F 3 "" H 6650 2050 60  0000 C CNN
 	1    6650 2050
@@
 F 0 "R34" H 4150 2200 50  0000 C CNN
 F 1 "820" H 4550 2200 50  0000 C CNN
-F 2 "" H 4350 2150 60  0000 C CNN
+F 2 "" H 4350 2150 60  0001 C CNN
 F 3 "" H 4350 2150 60  0000 C CNN
 	1    4350 2150
@@
 F 0 "C37" H 4750 3100 50  0000 L CNN
 F 1 "470pF" H 4750 2900 50  0000 L CNN
-F 2 "" H 4700 3000 60  0000 C CNN
+F 2 "" H 4700 3000 60  0001 C CNN
 F 3 "" H 4700 3000 60  0000 C CNN
 	1    4700 3000
@@
 $EndComp
 $Comp
-L GND #PWR087
+L GND #PWR100
 U 1 1 5A4A0477
 P 4700 3400
-F 0 "#PWR087" H 4700 3400 30  0001 C CNN
+F 0 "#PWR100" H 4700 3400 30  0001 C CNN
 F 1 "GND" H 4700 3330 30  0001 C CNN
 F 2 "" H 4700 3400 60  0000 C CNN
@@
 F 0 "C36" V 3600 2250 50  0000 L CNN
 F 1 "1500pF" V 3600 1800 50  0000 L CNN
-F 2 "" H 3550 2150 60  0000 C CNN
+F 2 "" H 3550 2150 60  0001 C CNN
 F 3 "" H 3550 2150 60  0000 C CNN
 	1    3550 2150
@@
 F 0 "R31" H 2700 2000 50  0000 C CNN
 F 1 "10k" H 3100 2000 50  0000 C CNN
-F 2 "" H 2900 1950 60  0000 C CNN
+F 2 "" H 2900 1950 60  0001 C CNN
 F 3 "" H 2900 1950 60  0000 C CNN
 	1    2900 1950
@@
 F 0 "R35" H 2700 2400 50  0000 C CNN
 F 1 "10k" H 3100 2400 50  0000 C CNN
-F 2 "" H 2900 2350 60  0000 C CNN
+F 2 "" H 2900 2350 60  0001 C CNN
 F 3 "" H 2900 2350 60  0000 C CNN
 	1    2900 2350
@@
 F 0 "R36" V 3800 3000 50  0000 C CNN
 F 1 "7.5K" V 4200 3050 50  0000 C CNN
-F 2 "" H 4000 2950 60  0000 C CNN
+F 2 "" H 4000 2950 60  0001 C CNN
 F 3 "" H 4000 2950 60  0000 C CNN
 	1    4000 2950
@@
 Connection ~ 4000 2350
 $Comp
-L GND #PWR088
+L GND #PWR99
 U 1 1 5A4A0BAE
 P 4000 3400
-F 0 "#PWR088" H 4000 3400 30  0001 C CNN
+F 0 "#PWR99" H 4000 3400 30  0001 C CNN
 F 1 "GND" H 4000 3330 30  0001 C CNN
 F 2 "" H 4000 3400 60  0000 C CNN
@@
 	4000 3400 4000 3150
 $Comp
-L OPA1664 U9
+L OPA1664 U8
 U 4 1 5A4A115F
 P 5300 5000
-F 0 "U9" H 5350 5200 60  0000 C CNN
+F 0 "U8" H 5350 5200 60  0000 C CNN
 F 1 "OPA1664" H 5450 4800 50  0000 C CNN
-F 2 "" H 5300 5000 60  0000 C CNN
+F 2 "" H 5300 5000 60  0001 C CNN
 F 3 "" H 5300 5000 60  0000 C CNN
 	4    5300 5000
@@
 	5200 4450 5200 4600
 $Comp
-L -5V #PWR089
+L -5V #PWR101
 U 1 1 5A4A1169
 P 6550 4450
-F 0 "#PWR089" H 6550 4590 20  0001 C CNN
+F 0 "#PWR101" H 6550 4590 20  0001 C CNN
 F 1 "-5V" H 6550 4560 30  0000 C CNN
 F 2 "" H 6550 4450 60  0000 C CNN
@@
 $EndComp
 $Comp
-L +5V #PWR090
+L +5V #PWR102
 U 1 1 5A4A116F
 P 6550 5600
-F 0 "#PWR090" H 6550 5690 20  0001 C CNN
+F 0 "#PWR102" H 6550 5690 20  0001 C CNN
 F 1 "+5V" H 6550 5690 30  0000 C CNN
 F 2 "" H 6550 5600 60  0000 C CNN
@@
 F 0 "C38" V 5250 4250 50  0000 L CNN
 F 1 "470pF" V 5250 3850 50  0000 L CNN
-F 2 "" H 5200 4150 60  0000 C CNN
+F 2 "" H 5200 4150 60  0001 C CNN
 F 3 "" H 5200 4150 60  0000 C CNN
 	1    5200 4150
@@
 F 0 "R37" H 5000 3850 50  0000 C CNN
 F 1 "7.5k" H 5400 3850 50  0000 C CNN
-F 2 "" H 5200 3800 60  0000 C CNN
+F 2 "" H 5200 3800 60  0001 C CNN
 F 3 "" H 5200 3800 60  0000 C CNN
 	1    5200 3800
@@
 F 0 "R39" H 4200 4950 50  0000 C CNN
 F 1 "820" H 4600 4950 50  0000 C CNN
-F 2 "" H 4400 4900 60  0000 C CNN
+F 2 "" H 4400 4900 60  0001 C CNN
 F 3 "" H 4400 4900 60  0000 C CNN
 	1    4400 4900
@@
 F 0 "R40" H 6500 5050 50  0000 C CNN
 F 1 "100" H 6900 5050 50  0000 C CNN
-F 2 "" H 6700 5000 60  0000 C CNN
+F 2 "" H 6700 5000 60  0001 C CNN
 F 3 "" H 6700 5000 60  0000 C CNN
 	1    6700 5000
@@
 F 0 "R41" H 4200 5150 50  0000 C CNN
 F 1 "820" H 4600 5150 50  0000 C CNN
-F 2 "" H 4400 5100 60  0000 C CNN
+F 2 "" H 4400 5100 60  0001 C CNN
 F 3 "" H 4400 5100 60  0000 C CNN
 	1    4400 5100
@@
 F 0 "C40" H 4800 6050 50  0000 L CNN
 F 1 "470pF" H 4800 5850 50  0000 L CNN
-F 2 "" H 4750 5950 60  0000 C CNN
+F 2 "" H 4750 5950 60  0001 C CNN
 F 3 "" H 4750 5950 60  0000 C CNN
 	1    4750 5950
@@
 $EndComp
 $Comp
-L GND #PWR091
+L GND #PWR104
 U 1 1 5A4A11CB
 P 4750 6350
-F 0 "#PWR091" H 4750 6350 30  0001 C CNN
+F 0 "#PWR104" H 4750 6350 30  0001 C CNN
 F 1 "GND" H 4750 6280 30  0001 C CNN
 F 2 "" H 4750 6350 60  0000 C CNN
@@
 F 0 "C39" V 3650 5200 50  0000 L CNN
 F 1 "1500pF" V 3650 4750 50  0000 L CNN
-F 2 "" H 3600 5100 60  0000 C CNN
+F 2 "" H 3600 5100 60  0001 C CNN
 F 3 "" H 3600 5100 60  0000 C CNN
 	1    3600 5100
@@
 F 0 "R38" H 2750 4950 50  0000 C CNN
 F 1 "10k" H 3150 4950 50  0000 C CNN
-F 2 "" H 2950 4900 60  0000 C CNN
+F 2 "" H 2950 4900 60  0001 C CNN
 F 3 "" H 2950 4900 60  0000 C CNN
 	1    2950 4900
@@
 F 0 "R42" H 2750 5350 50  0000 C CNN
 F 1 "10k" H 3150 5350 50  0000 C CNN
-F 2 "" H 2950 5300 60  0000 C CNN
+F 2 "" H 2950 5300 60  0001 C CNN
 F 3 "" H 2950 5300 60  0000 C CNN
 	1    2950 5300
@@
 F 0 "R43" V 3850 5950 50  0000 C CNN
 F 1 "7.5K" V 4250 6000 50  0000 C CNN
-F 2 "" H 4050 5900 60  0000 C CNN
+F 2 "" H 4050 5900 60  0001 C CNN
 F 3 "" H 4050 5900 60  0000 C CNN
 	1    4050 5900
@@
 Connection ~ 4050 5300
 $Comp
-L GND #PWR092
+L GND #PWR103
 U 1 1 5A4A1201
 P 4050 6350
-F 0 "#PWR092" H 4050 6350 30  0001 C CNN
+F 0 "#PWR103" H 4050 6350 30  0001 C CNN
 F 1 "GND" H 4050 6280 30  0001 C CNN
 F 2 "" H 4050 6350 60  0000 C CNN
