File: audio_input.sch (KiCad schematic (older format))
At the start: 15 parts, among them U8 OPA1664

Commit message: Added more footprint associations, added new footprints to lib
Parts:
- R24, R25, R26, R27, R28, R29: footprint (none) -> Resistors_SMD:R_0805_HandSoldering
Changed lines of the file:
@@
 F 0 "R24" H 4800 950 50  0000 C CNN
 F 1 "10k,5%" H 5250 950 50  0000 C CNN
-F 2 "" H 5000 900 60  0001 C CNN
+F 2 "Resistors_SMD:R_0805_HandSoldering" H 5000 900 60  0001 C CNN
 F 3 "" H 5000 900 60  0000 C CNN
 	1    5000 900
@@
 F 0 "R25" H 3900 2050 50  0000 C CNN
 F 1 "20k,1%" H 4350 2050 50  0000 C CNN
-F 2 "" H 4100 2000 60  0001 C CNN
+F 2 "Resistors_SMD:R_0805_HandSoldering" H 4100 2000 60  0001 C CNN
 F 3 "" H 4100 2000 60  0000 C CNN
 	1    4100 2000
@@
 F 0 "R26" H 6300 2150 50  0000 C CNN
 F 1 "1k,1%" H 6700 2150 50  0000 C CNN
-F 2 "" H 6500 2100 60  0001 C CNN
+F 2 "Resistors_SMD:R_0805_HandSoldering" H 6500 2100 60  0001 C CNN
 F 3 "" H 6500 2100 60  0000 C CNN
 	1    6500 2100
@@
 F 0 "R27" H 4800 3900 50  0000 C CNN
 F 1 "10k,5%" H 5250 3900 50  0000 C CNN
-F 2 "" H 5000 3850 60  0001 C CNN
+F 2 "Resistors_SMD:R_0805_HandSoldering" H 5000 3850 60  0001 C CNN
 F 3 "" H 5000 3850 60  0000 C CNN
 	1    5000 3850
@@
 F 0 "R28" H 3900 5000 50  0000 C CNN
 F 1 "20k,1%" H 4350 5000 50  0000 C CNN
-F 2 "" H 4100 4950 60  0001 C CNN
+F 2 "Resistors_SMD:R_0805_HandSoldering" H 4100 4950 60  0001 C CNN
 F 3 "" H 4100 4950 60  0000 C CNN
 	1    4100 4950
@@
 F 0 "R29" H 6300 5100 50  0000 C CNN
 F 1 "1k,1%" H 6700 5100 50  0000 C CNN
-F 2 "" H 6500 5050 60  0001 C CNN
+F 2 "Resistors_SMD:R_0805_HandSoldering" H 6500 5050 60  0001 C CNN
 F 3 "" H 6500 5050 60  0000 C CNN
 	1    6500 5050

Commit message: Added lib parts, adding atmega32u4 to board schematic, adding new CODED crystal
Parts:
- removed JP1: JUMPER3, Pin_Headers:Pin_Header_Straight_1x03, symbol JUMPER3
- added C?: 0.1uF, Capacitors_THT:C_Rect_L18_W11_H19_P15, symbol C
- added C?: 10uF, Capacitors_THT:C_Rect_L18_W11_H19_P15, symbol C
- added R? (x2): 10k,0.5%, symbol R
- C29: value 330pF,2.5% -> 3.3nF,2.5%
- C30, C33: symbol CP1 -> C; Type (none) -> Film
- R24: value 10k,5% -> 1k,5%
- R25: value 20k,1% -> 2k,1%
Connections:
- net +5V: now also R?.2
- net GND: now also U8.11 (V-), C?.2, C?.2, R?.1
- net at C30.1, R25.2: now also C?.1, C?.1, R?.1, R?.2
Other:
- note added: "Rail-to-rail operation will not damage ADC; \nno protection needed.\n\nVBIAS @ 2.5V no distortion expected."
- note removed: "If op-amp is grounded, rail-to-rail operation\nwill not damage ADC; no protection needed.\nStudy sound quality effects.\n\nVBIAS @ 2.5V no distortion expected."
Changed lines of the file:
@@
 LIBS:muse_mini
 LIBS:musev2
+LIBS:autodrive
+LIBS:atx24
+LIBS:musev3-cache
 EELAYER 25 0
 EELAYER END
@@
 $EndComp
 $Comp
-L -5V #PWR089
-U 1 1 5A49B7EA
-P 6450 1250
-F 0 "#PWR089" H 6450 1390 20  0001 C CNN
-F 1 "-5V" H 6450 1360 30  0000 C CNN
-F 2 "" H 6450 1250 60  0000 C CNN
-F 3 "" H 6450 1250 60  0000 C CNN
-	1    6450 1250
-	1    0    0    -1
-$EndComp
-$Comp
 L C C29
 U 1 1 5A49B886
 P 5000 1250
 F 0 "C29" V 5050 1350 50  0000 L CNN
-F 1 "330pF,2.5%" V 5050 750 50  0000 L CNN
+F 1 "3.3nF,2.5%" V 5050 750 50  0000 L CNN
 F 2 "muse-v3:C_Rect_L7.2_W4.5_P5" H 5000 1250 60  0001 C CNN
 F 3 "" H 5000 1250 60  0000 C CNN
@@
 P 5000 900
 F 0 "R24" H 4800 950 50  0000 C CNN
-F 1 "10k,5%" H 5250 950 50  0000 C CNN
+F 1 "1k,5%" H 5250 950 50  0000 C CNN
 F 2 "Resistors_SMD:R_0805_HandSoldering" H 5000 900 60  0001 C CNN
 F 3 "" H 5000 900 60  0000 C CNN
@@
 P 4100 2000
 F 0 "R25" H 3900 2050 50  0000 C CNN
-F 1 "20k,1%" H 4350 2050 50  0000 C CNN
+F 1 "2k,1%" H 4350 2050 50  0000 C CNN
 F 2 "Resistors_SMD:R_0805_HandSoldering" H 4100 2000 60  0001 C CNN
 F 3 "" H 4100 2000 60  0000 C CNN
@@
 	1    0    0    -1
 $EndComp
-Text HLabel 3250 2000 0    60   Input ~ 0
+Text HLabel 2150 2000 0    60   Input ~ 0
 AUDIO_IN_L
 Text HLabel 7550 2100 2    60   Input ~ 0
@@
 L +5V #PWR093
 U 1 1 5A49B806
-P 6350 2550
-F 0 "#PWR093" H 6350 2640 20  0001 C CNN
-F 1 "+5V" H 6350 2640 30  0000 C CNN
-F 2 "" H 6350 2550 60  0000 C CNN
-F 3 "" H 6350 2550 60  0000 C CNN
-	1    6350 2550
-	0    1    1    0
+P 5150 2550
+F 0 "#PWR093" H 5150 2640 20  0001 C CNN
+F 1 "+5V" H 5150 2640 30  0000 C CNN
+F 2 "" H 5150 2550 60  0000 C CNN
+F 3 "" H 5150 2550 60  0000 C CNN
+	1    5150 2550
+	1    0    0    -1
 $EndComp
 Text Notes 1100 1200 0    60   ~ 0
 2-Vrms Input\nG: 0.5\nFc: 48 kHz
 Wire Wire Line
-	3250 2000 3400 2000
+	2150 2000 2300 2000
 Wire Wire Line
 	4300 2000 4600 2000
@@
 	4350 2200 4600 2200
 Wire Wire Line
-	5000 1550 6350 1550
+	5000 1550 5150 1550
 Wire Wire Line
 	5600 2100 6300 2100
@@
 Wire Wire Line
 	4350 3450 4350 3250
-Wire Wire Line
-	3900 2000 3800 2000
 Connection ~ 5700 2100
 Wire Wire Line
@@
 Connection ~ 5700 5050
 Wire Wire Line
-	5000 2550 6350 2550
-Wire Wire Line
-	5000 2550 5000 2500
+	5000 2600 5150 2600
+Wire Wire Line
+	5000 2600 5000 2500
 Wire Wire Line
 	5000 5500 5000 5450
@@
 48.2+/-3.4 kHz Low-Pass Filter
 $Comp
-L CP1 C33
+L C C33
 U 1 1 5A49EA97
 P 3600 4950
 F 0 "C33" V 3550 4750 50  0000 L CNN
-F 1 "10uF" V 3700 5050 50  0000 L CNN
+F 1 "10uF" V 3650 5000 50  0000 L CNN
 F 2 "Capacitors_SMD:c_elec_6.3x5.7" H 3600 4950 60  0001 C CNN
 F 3 "" H 3600 4950 60  0000 C CNN
+F 4 "Film" V 3650 4900 60  0000 R CNN "Type"
 	1    3600 4950
 	0    1    1    0
 $EndComp
 $Comp
-L CP1 C30
+L C C30
 U 1 1 5A49B8DC
-P 3600 2000
-F 0 "C30" V 3550 1800 50  0000 L CNN
-F 1 "10uF" V 3700 2100 50  0000 L CNN
-F 2 "Capacitors_SMD:c_elec_6.3x5.7" H 3600 2000 60  0001 C CNN
-F 3 "" H 3600 2000 60  0000 C CNN
-	1    3600 2000
-	0    1    1    0
-$EndComp
-$Comp
-L JUMPER3 JP1
-U 1 1 5A4F87E9
-P 6450 1550
-F 0 "JP1" H 6500 1450 40  0000 L CNN
-F 1 "JUMPER3" H 6450 1650 40  0000 C CNN
-F 2 "Pin_Headers:Pin_Header_Straight_1x03" H 6450 1550 60  0001 C CNN
-F 3 "" H 6450 1550 60  0000 C CNN
-	1    6450 1550
-	0    1    1    0
-$EndComp
-Wire Wire Line
-	6450 1300 6450 1250
+P 2500 2000
+F 0 "C30" V 2450 1800 50  0000 L CNN
+F 1 "10uF" V 2550 2050 50  0000 L CNN
+F 2 "Capacitors_SMD:c_elec_6.3x5.7" H 2500 2000 60  0001 C CNN
+F 3 "" H 2500 2000 60  0000 C CNN
+F 4 "Film" V 2550 1950 60  0000 R CNN "Type"
+	1    2500 2000
+	0    1    1    0
+$EndComp
 $Comp
 L GND #PWR094
 U 1 1 5A4F89F7
-P 6450 1850
-F 0 "#PWR094" H 6450 1850 30  0001 C CNN
-F 1 "GND" H 6450 1780 30  0001 C CNN
-F 2 "" H 6450 1850 60  0000 C CNN
-F 3 "" H 6450 1850 60  0000 C CNN
-	1    6450 1850
-	1    0    0    -1
-$EndComp
-Wire Wire Line
-	6450 1850 6450 1800
-Text Notes 6650 1800 0    60   ~ 0
-If op-amp is grounded, rail-to-rail operation\nwill not damage ADC; no protection needed.\nStudy sound quality effects.\n\nVBIAS @ 2.5V no distortion expected.
+P 5150 1600
+F 0 "#PWR094" H 5150 1600 30  0001 C CNN
+F 1 "GND" H 5150 1530 30  0001 C CNN
+F 2 "" H 5150 1600 60  0000 C CNN
+F 3 "" H 5150 1600 60  0000 C CNN
+	1    5150 1600
+	1    0    0    -1
+$EndComp
+Wire Wire Line
+	5150 1550 5150 1600
+Text Notes 5800 1800 0    60   ~ 0
+Rail-to-rail operation will not damage ADC; \nno protection needed.\n\nVBIAS @ 2.5V no distortion expected.
 $Comp
 L -5V #PWR095
@@
 Wire Wire Line
 	6450 4800 6450 4750
+$Comp
+L R R?
+U 1 1 5B2B2643
+P 2850 2350
+F 0 "R?" V 2700 2400 50  0000 L CNN
+F 1 "10k,0.5%" V 3000 2400 50  0000 L CNN
+F 2 "" H 2850 2350 60  0000 C CNN
+F 3 "" H 2850 2350 60  0000 C CNN
+	1    2850 2350
+	0    1    1    0
+$EndComp
+Wire Wire Line
+	2700 2000 3900 2000
+Wire Wire Line
+	2850 1850 2850 2150
+Connection ~ 2850 2000
+$Comp
+L C C?
+U 1 1 5B2B2A01
+P 3400 2350
+F 0 "C?" H 3450 2500 50  0000 L CNN
+F 1 "0.1uF" H 3450 2200 50  0000 L CNN
+F 2 "Capacitors_THT:C_Rect_L18_W11_H19_P15" H 3400 2350 60  0001 C CNN
+F 3 "" H 3400 2350 60  0000 C CNN
+	1    3400 2350
+	1    0    0    -1
+$EndComp
+Wire Wire Line
+	3400 2150 3400 2000
+Connection ~ 3400 2000
+$Comp
+L GND #PWR?
+U 1 1 5B2B2B32
+P 2850 2650
+F 0 "#PWR?" H 2850 2650 30  0001 C CNN
+F 1 "GND" H 2850 2580 30  0001 C CNN
+F 2 "" H 2850 2650 60  0000 C CNN
+F 3 "" H 2850 2650 60  0000 C CNN
+	1    2850 2650
+	1    0    0    -1
+$EndComp
+Wire Wire Line
+	2850 2550 2850 2650
+$Comp
+L GND #PWR?
+U 1 1 5B2B2BC5
+P 3400 2650
+F 0 "#PWR?" H 3400 2650 30  0001 C CNN
+F 1 "GND" H 3400 2580 30  0001 C CNN
+F 2 "" H 3400 2650 60  0000 C CNN
+F 3 "" H 3400 2650 60  0000 C CNN
+	1    3400 2650
+	1    0    0    -1
+$EndComp
+Wire Wire Line
+	3400 2650 3400 2550
+$Comp
+L +5V #PWR?
+U 1 1 5B2B2CA5
+P 2850 1350
+F 0 "#PWR?" H 2850 1440 20  0001 C CNN
+F 1 "+5V" H 2850 1440 30  0000 C CNN
+F 2 "" H 2850 1350 60  0000 C CNN
+F 3 "" H 2850 1350 60  0000 C CNN
+	1    2850 1350
+	1    0    0    -1
+$EndComp
+Wire Wire Line
+	2850 1450 2850 1350
+Wire Wire Line
+	5150 2600 5150 2550
+$Comp
+L R R?
+U 1 1 5B2B3ADD
+P 2850 1650
+F 0 "R?" V 2700 1700 50  0000 L CNN
+F 1 "10k,0.5%" V 3000 1700 50  0000 L CNN
+F 2 "" H 2850 1650 60  0000 C CNN
+F 3 "" H 2850 1650 60  0000 C CNN
+	1    2850 1650
+	0    1    1    0
+$EndComp
+$Comp
+L C C?
+U 1 1 5B2B42CB
+P 3700 2350
+F 0 "C?" H 3750 2500 50  0000 L CNN
+F 1 "10uF" H 3750 2200 50  0000 L CNN
+F 2 "Capacitors_THT:C_Rect_L18_W11_H19_P15" H 3700 2350 60  0001 C CNN
+F 3 "" H 3700 2350 60  0000 C CNN
+	1    3700 2350
+	1    0    0    -1
+$EndComp
+Wire Wire Line
+	3700 2150 3700 2000
+Connection ~ 3700 2000
+$Comp
+L GND #PWR?
+U 1 1 5B2B43E4
+P 3700 2650
+F 0 "#PWR?" H 3700 2650 30  0001 C CNN
+F 1 "GND" H 3700 2580 30  0001 C CNN
+F 2 "" H 3700 2650 60  0000 C CNN
+F 3 "" H 3700 2650 60  0000 C CNN
+	1    3700 2650
+	1    0    0    -1
+$EndComp
+Wire Wire Line
+	3700 2650 3700 2550
 $EndSCHEMATC
