File: musev3.sch (KiCad schematic (older format))
At the start: 82 parts, among them CON1 RCA_conn_x2, CON2 3.5mm_conn_tip_switch, CON3 3.5mm_conn_tip_switch, J1 RJ45-TRANSFO, P1 PWR_IN_PINS, P2 RF_DEBUG, P3 LED_CONN, P4 UART_CONN, P5 SMA, SW1 UART_DEBUG, SW2 RST, U1 74HC04, U2 R1171S331B, U3 GTL2010, U4 onion_omega2, U5 LM2662, U6 PCM3060, U7 RFM69HCW, X1 CFPS-73 - 24.567MHz

Commit message: Added more footprint assoc. & eth. pulldown resistors
Parts:
- removed J1: RJ45-TRANSFO, symbol RJ45-TRANSFO
- removed JP1: JUMPER, symbol JUMPER
- added C49, C50: 100nF, Capacitors_SMD:C_0805_HandSoldering, symbol C
- added J1: RJMG163128101NR, muse-v3:RJMG163128101NR, symbol RJMG163128101NR
- added R44, R45, R46, R47: 49.9,1%, symbol R
- C22, C25: footprint Capacitors_SMD:C_0805_HandSoldering -> muse-v3:C_Rect_L7.5_W6.5_P5
- CON1: footprint (none) -> muse-v2-lib:PJRAS2X2S01X
- CON2, CON3: footprint (none) -> muse-v2-lib:3.5MM-AUDIO-SMD
- D1: footprint (none) -> LEDs:LED-5MM
- D2: renamed from D6; footprint (none) -> TO_SOT_Packages_SMD:TSOT-6-MK06A_Handsoldering
- D3: renamed from D7; footprint (none) -> TO_SOT_Packages_SMD:TSOT-6-MK06A_Handsoldering
- P1: footprint (none) -> Pin_Headers:Pin_Header_Straight_1x03
- P2: footprint (none) -> Pin_Headers:Pin_Header_Straight_1x06
- P3: footprint (none) -> Pin_Headers:Pin_Header_Straight_1x10
- P4: footprint (none) -> Pin_Headers:Pin_Header_Angled_1x06
- R1, R10, R11, R12, R13, R14, R15, R16, R17, R18, R19, R2, R20, R21, R22, R23, R3, R4, R5, R6, R7, R8, R9: footprint (none) -> Resistors_SMD:R_0805_HandSoldering
Connections:
- wire segments 355 -> 471
Other:
- note added: "What connector\nshould we use?"
- moved on the sheet: C14, D1, R1

Commit message: Added more footprint associations, added new footprints to lib
Parts:
- R44, R45, R46, R47: footprint (none) -> Resistors_SMD:R_0805_HandSoldering
- SW1: footprint (none) -> muse-v3:JS202011CQN
- SW2: footprint (none) -> muse-v3:FSM4JH
- U1: footprint (none) -> Housings_SOIC:SOIC-14_3.9x8.7mm_Pitch1.27mm

Commit message: Added lib parts, adding atmega32u4 to board schematic, adding new CODED crystal
Parts:
- removed C10, C9: 4.7uF, Capacitors_SMD:C_0805_HandSoldering, symbol CP1
- removed C15, C24, C26: 47uF, Capacitors_SMD:c_elec_5x5.3, symbol CP1
- removed C20: 1uF, Capacitors_SMD:C_0805_HandSoldering, symbol CP1
- removed C21: 100nF, Capacitors_SMD:C_0805_HandSoldering, symbol C
- removed C43, C44, C6, C8: 0.1uF, Capacitors_SMD:C_0805_HandSoldering, symbol C
- removed C5, C7: 10uF, Capacitors_SMD:c_elec_6.3x5.7, symbol CP1
- removed P1: PWR_IN_PINS, Pin_Headers:Pin_Header_Straight_1x03, symbol PWR_IN_PINS
- removed P2: RF_DEBUG, Pin_Headers:Pin_Header_Straight_1x06, symbol CONN_01X06
- removed P5: SMA, symbol BNC
- removed unit 1 of U1
- removed unit 2 of U1
- removed unit 6 of U1
- removed U2: R1171S331B, symbol R1171S331B
- removed U5: LM2662, symbol LM2662
- removed U7: RFM69HCW, symbol RFM69HCW
- added D?: PWR_LED, LEDs:LED-5MM, symbol LED
- added J?: ATX24, symbol ATX24
- added R? (x2): 10k,0.5%, symbol R
- added R?: 160, Resistors_SMD:R_0805_HandSoldering, symbol R
- added U?: ATMEGA32U4-A, TQFP44, symbol ATMEGA32U4-A
- R1: value 4.7k -> 160
Connections:
- net +3.3V: now also J?.1 (3V3), J?.12 (3V3), J?.13 (3V3), J?.2 (3V3); no longer R1.2
- net +5V: now also R1.2, J?.21 (5V), J?.22 (5V), J?.23 (5V), J?.4 (5V), J?.6 (5V), R?.2
- net -5V: now also J?.20 (-5V)
- net CODEC_VCOM: now also R?.1, R?.2
- net GND: now also D?.2 (K), J?.15 (GND), J?.17 (GND), J?.18 (GND), J?.19 (GND), J?.24 (GND), J?.3 (GND), J?.5 (GND), J?.7 (GND), R?.1; no longer U4.32 (GND)
- net SPI_CS: now also U6.27 (~MS~/ADR/IFMD)
- net USB_D-: now reaches U4.29 (USB_D-)
- net USB_D+: now reaches U4.30 (USB_D+)
- net RF_DATA: no longer names the net of U4.17 (GPIO_5/I2C_SDA)
- net RF_DCLK: no longer names the net of U4.18 (GPIO_4/I2C_SCL)
- new net: D?.1 (A), R?.1
- new net +12V: J?.10 (12V), J?.11 (12V)
- new net +5VSB: J?.9 (5VSB), R?.2
- new net -12V: J?.14 (-12)
- new net PS_ON: J?.16 (PS_ON)
- new net PWR_OK: J?.8 (POK)
- no-connect marks 15 -> 14
Other:
- note added: "Audio Input/Output Filters"
- note removed: "Are more power inputs required?\nHow is the relay wired? Do we have a standby PSU?"
- note removed: "Audio Input/Output Buffers"
- note removed: "CODEC Selected when \nRF is disconnected"
- note removed: "DIO Tx - MODE: Continous 00\n0 -> PllLock\n1 -> DCLK\n2 -> DATA\n3 -> TxReady\n4 -> TxReady\n5 -> CLKOUT"
- note removed: "FC = V+ for \n150kHz F_OSC"
- note removed: "FM Radio"
- note removed: "FM Radio Pin Breakout"
- note removed: "LV = GND for\nV+ > 3.5V"
- note removed: "Low Drop-Out Regulator"
- note removed: "NOTE: Capacitors must have ESR < 0.2 Ohm"
- note removed: "Voltage Inverter"
- note removed: "What connector\nshould we use?"
- moved on the sheet: C1, C11, C12, C13, C14, C16, C17, C18, C19, C2, C22, C23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

Commit message: upgraded to kicad v5.0
Parts:
- C1, C11, C14, C16, C19, C28, C3: symbol CP1 -> device:CP1
- C12, C17, C18, C2, C22, C23, C25, C27, C4, C41, C42, C45, C46, C47, C48, C49, C50: symbol C -> Solar-Car-Components:C
- C13: symbol C-RESCUE-museV2 -> musev2:C-RESCUE-museV2
- CON1: symbol RCA_conn_x2 -> musev2:RCA_conn_x2
- CON2, CON3: symbol 3.5mm_conn_tip_switch -> musev2:3.5mm_conn_tip_switch
- D1, D?: symbol LED -> Solar-Car-Components:LED
- D2, D3: symbol TPD2E1B06 -> musev3:TPD2E1B06
- J1: symbol RJMG163128101NR -> musev3:RJMG163128101NR
- J?: symbol ATX24 -> atx24:ATX24
- P3: symbol CONN_01X10 -> conn:CONN_01X10
- P4: symbol CONN_01X06 -> conn:CONN_01X06
- R1, R10, R11, R12, R13, R14, R15, R16, R17, R18, R19, R2, R20, R21, R22, R23, R3, R4, R44, R45, R46, R47, R5, R6, R7, R8, R9, R? (x3): symbol R -> Solar-Car-Components:R
- SW1: symbol DUAL_SWITCH_INV -> device:DUAL_SWITCH_INV
- SW2: symbol DPST -> device:DPST
- U1: symbol 74HC04 -> 74xx1:74HC04
- U3: symbol GTL2010 -> musev2:GTL2010
- U4: symbol onion_omega2 -> musev3:onion_omega2
- U6: symbol PCM3060 -> muse_mini:PCM3060
- U?: symbol ATMEGA32U4-A -> atmel:ATMEGA32U4-A
- X1: symbol CFPS-73 -> muse_mini:CFPS-73
Connections:
- net +5V: no longer J?.21 (5V)
